File: lidar_pcb/lidar_pcb.kicad_sch (KiCad schematic)
At the start: 28 parts, among them J2 Conn_01x02, J3 Conn_01x07, U1 VL53L9CXV0VE_1, U2 TLV62568PDRLT, U3 TLV62568PDRLT, U4 TXB0104RGYRG4, U5 TXB0102DCUR

Commit message: Opraveni README, aby tam bylo vse ke kontrole
Connections:
- net AVDD: no longer C1.2, C10.2, C11.2, C12.2, C13.2, C14.2, C15.2, C2.1, C2.2, C3.2, C5.1, C5.2, C7.2, C8.2, C9.2, J2.1 (Pin_1), J2.2 (Pin_2), J3.3 (Pin_3), R2.2, R4.2, U1.A1 (VSS), U1.A2 (VSS_DRIVER), U1.A3 (VSS_DRIVER), U1.A4 (VSS), U1.A7 (VSS), U1.B4 (VSS), U1.B5 (VSS), U1.B6 (VSS), U1.B7 (VSS), U1.B8 (VSS), U1.B9 (VSS), U1.C1 (VSS), U1.D4 (VSS), U1.D5 (VSS), U1.D6 (VSS), U1.D7 (VSS), U1.D8 (VSS), U1.D9 (VSS), U1.E1 (VSS), U1.E10 (VSS), U1.E2 (VSS), U1.E4 (VSS), U1.E5 (VSS), U1.E9 (VSS), U2.2 (GND), U2.3 (VIN), U2.5 (EN), U3.2 (GND), U3.3 (VIN), U3.5 (EN), U4.15 (EXP), U4.7 (GND), U5.2 (GND)
- new net 5V: C2.1, C5.1, J2.2 (Pin_2), U2.3 (VIN), U2.5 (EN), U3.3 (VIN), U3.5 (EN)
- new net GND: C1.2, C10.2, C11.2, C12.2, C13.2, C14.2, C15.2, C2.2, C3.2, C5.2, C7.2, C8.2, C9.2, J2.1 (Pin_1), J3.3 (Pin_3), R2.2, R4.2, U1.A1 (VSS), U1.A2 (VSS_DRIVER), U1.A3 (VSS_DRIVER), U1.A4 (VSS), U1.A7 (VSS), U1.B4 (VSS), U1.B5 (VSS), U1.B6 (VSS), U1.B7 (VSS), U1.B8 (VSS), U1.B9 (VSS), U1.C1 (VSS), U1.D4 (VSS), U1.D5 (VSS), U1.D6 (VSS), U1.D7 (VSS), U1.D8 (VSS), U1.D9 (VSS), U1.E1 (VSS), U1.E10 (VSS), U1.E2 (VSS), U1.E4 (VSS), U1.E5 (VSS), U1.E9 (VSS), U2.2 (GND), U3.2 (GND), U4.15 (EXP), U4.7 (GND), U5.2 (GND)
Other:
- moved on the sheet: C11, C5
Changed lines of the file:
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@@
 	)
 	(junction
-		(at 270.51 85.09)
-		(diameter 0)
-		(color 0 0 0 0)
-	)
-	(junction
 		(at 104.14 82.55)
 		(diameter 0)
@@
 	)
 	(junction
-		(at 34.29 105.41)
-		(diameter 0)
-		(color 0 0 0 0)
-	)
-	(junction
 		(at 93.98 82.55)
 		(diameter 0)
@@
 	)
 	(junction
-		(at 34.29 104.14)
+		(at 248.92 67.31)
 		(diameter 0)
 		(color 0 0 0 0)
 	)
 	(junction
-		(at 248.92 67.31)
+		(at 176.53 114.3)
 		(diameter 0)
 		(color 0 0 0 0)
 	)
 	(junction
-		(at 176.53 114.3)
+		(at 273.05 76.2)
 		(diameter 0)
 		(color 0 0 0 0)
@@
 	)
 	(junction
+		(at 130.81 49.53)
+		(diameter 0)
+		(color 0 0 0 0)
+	)
+	(junction
 		(at 265.43 81.28)
 		(diameter 0)
@@
 	)
 	(junction
-		(at 270.51 76.2)
-		(diameter 0)
-		(color 0 0 0 0)
-	)
-	(junction
 		(at 99.06 55.88)
 		(diameter 0)
@@
 	)
 	(junction
-		(at 270.51 77.47)
+		(at 129.54 123.19)
 		(diameter 0)
 		(color 0 0 0 0)
@@
 	(wire
 		(pts
-			(xy 34.29 105.41) (xy 34.29 113.03)
+			(xy 180.34 121.92) (xy 180.34 123.19)
 		)
 		(stroke
@@
 	(wire
 		(pts
-			(xy 180.34 121.92) (xy 180.34 123.19)
+			(xy 34.29 109.22) (xy 34.29 106.68)
 		)
 		(stroke
@@
 	(wire
 		(pts
-			(xy 27.94 34.29) (xy 40.64 34.29)
+			(xy 129.54 120.65) (xy 129.54 123.19)
 		)
 		(stroke
@@
 	(wire
 		(pts
-			(xy 176.53 133.35) (xy 186.69 133.35)
+			(xy 27.94 34.29) (xy 40.64 34.29)
 		)
 		(stroke
@@
 	(wire
 		(pts
-			(xy 34.29 92.71) (xy 34.29 104.14)
+			(xy 176.53 133.35) (xy 186.69 133.35)
 		)
 		(stroke
@@
 	(wire
 		(pts
-			(xy 270.51 77.47) (xy 270.51 76.2)
+			(xy 273.05 77.47) (xy 273.05 76.2)
 		)
 		(stroke
@@
 	(wire
 		(pts
-			(xy 34.29 104.14) (xy 34.29 105.41)
-		)
-		(stroke
-			(width 0)
-			(type default)
-		)
-	)
-	(wire
-		(pts
 			(xy 177.8 44.45) (xy 177.8 46.99)
 		)
@@
 	(wire
 		(pts
-			(xy 130.81 49.53) (xy 142.24 49.53)
-		)
-		(stroke
-			(width 0)
-			(type default)
-		)
-	)
-	(wire
-		(pts
 			(xy 177.8 69.85) (xy 184.15 69.85)
 		)
@@
 	(wire
 		(pts
-			(xy 270.51 85.09) (xy 270.51 86.36)
+			(xy 273.05 85.09) (xy 273.05 86.36)
 		)
 		(stroke
@@
 	(wire
 		(pts
-			(xy 265.43 76.2) (xy 270.51 76.2)
+			(xy 265.43 76.2) (xy 273.05 76.2)
 		)
 		(stroke
@@
 	(wire
 		(pts
-			(xy 270.51 62.23) (xy 270.51 76.2)
+			(xy 273.05 62.23) (xy 273.05 76.2)
 		)
 		(stroke
@@
 	(wire
 		(pts
-			(xy 270.51 77.47) (xy 270.51 85.09)
+			(xy 130.81 46.99) (xy 130.81 49.53)
 		)
 		(stroke
@@
 	(wire
 		(pts
+			(xy 130.81 49.53) (xy 142.24 49.53)
+		)
+		(stroke
+			(width 0)
+			(type default)
+		)
+	)
+	(wire
+		(pts
+			(xy 34.29 92.71) (xy 34.29 99.06)
+		)
+		(stroke
+			(width 0)
+			(type default)
+		)
+	)
+	(wire
+		(pts
 			(xy 110.49 29.21) (xy 110.49 38.1)
 		)
@@
 	)
 	(label "3.3V"
-		(at 130.81 49.53 0)
+		(at 130.81 46.99 0)
 		(fields_autoplaced yes)
 		(effects
@@
 	)
 	(label "3.3V"
-		(at 129.54 123.19 0)
+		(at 129.54 120.65 0)
 		(fields_autoplaced yes)
 		(effects
@@
 	)
 	(label "3.3V"
-		(at 270.51 62.23 0)
+		(at 273.05 62.23 0)
 		(fields_autoplaced yes)
 		(effects
@@
 	(symbol
 		(lib_id "Device:C")
-		(at 34.29 109.22 0)
+		(at 34.29 102.87 0)
 		(unit 1)
 		(exclude_from_sim no)
@@
 		(dnp no)
 		(property "Reference" "C5"
-			(at 35.56 96.266 0)
+			(at 34.798 100.33 0)
 			(effects
 				(font
@@
 		)
 		(property "Value" "4.7u"
-			(at 34.798 101.346 0)
+			(at 34.544 105.41 0)
 			(effects
 				(font
@@
 		)
 		(property "Footprint" "Capacitor_SMD:C_0805_2012Metric"
-			(at 35.2552 113.03 0)
+			(at 35.2552 106.68 0)
 			(effects
 				(font
@@
 		)
 		(property "Datasheet" "~"
-			(at 34.29 109.22 0)
+			(at 34.29 102.87 0)
 			(effects
 				(font
@@
 		)
 		(property "Description" "Unpolarized capacitor"
-			(at 34.29 109.22 0)
+			(at 34.29 102.87 0)
 			(effects
 				(font
@@
 	(symbol
 		(lib_id "power:GND")
-		(at 270.51 86.36 0)
+		(at 273.05 86.36 0)
 		(unit 1)
 		(exclude_from_sim no)
@@
 		(fields_autoplaced yes)
 		(property "Reference" "#PWR014"
-			(at 270.51 92.71 0)
+			(at 273.05 92.71 0)
 			(effects
 				(font
@@
 		)
 		(property "Value" "GND"
-			(at 270.51 91.44 0)
+			(at 273.05 91.44 0)
 			(effects
 				(font
@@
 		)
 		(property "Footprint" ""
-			(at 270.51 86.36 0)
+			(at 273.05 86.36 0)
 			(effects
 				(font
@@
 		)
 		(property "Datasheet" ""
-			(at 270.51 86.36 0)
+			(at 273.05 86.36 0)
 			(effects
 				(font
@@
 		)
 		(property "Description" "Power symbol creates a global label with name \"GND\" , ground"
-			(at 270.51 86.36 0)
+			(at 273.05 86.36 0)
 			(effects
 				(font
@@
 	(symbol
 		(lib_id "Device:C")
-		(at 270.51 81.28 0)
+		(at 273.05 81.28 0)
 		(unit 1)
 		(exclude_from_sim no)
@@
 		(dnp no)
 		(property "Reference" "C11"
-			(at 270.764 78.74 0)
+			(at 273.304 78.74 0)
 			(effects
 				(font
@@
 		)
 		(property "Value" "4.7u"
-			(at 271.78 83.566 0)
+			(at 274.32 83.566 0)
 			(effects
 				(font
@@
 		)
 		(property "Footprint" "Capacitor_SMD:C_0805_2012Metric"
-			(at 271.4752 85.09 0)
+			(at 274.0152 85.09 0)
 			(effects
 				(font
@@
 		)
 		(property "Datasheet" "~"
-			(at 270.51 81.28 0)
+			(at 273.05 81.28 0)
 			(effects
 				(font
@@
 		)
 		(property "Description" "Unpolarized capacitor"
-			(at 270.51 81.28 0)
+			(at 273.05 81.28 0)
 			(effects
 				(font
@@
 		(on_board yes)
 		(dnp no)
-		(fields_autoplaced yes)
 		(property "Reference" "C13"
-			(at 184.15 116.8399 0)
+			(at 182.118 115.824 0)
 			(effects
 				(font
@@
 		)
 		(property "Value" "0.1u"
-			(at 184.15 119.3799 0)
+			(at 181.61 120.65 0)
 			(effects
 				(font
@@
 	(symbol
 		(lib_id "power:GND")
-		(at 34.29 104.14 0)
+		(at 34.29 109.22 0)
 		(unit 1)
 		(exclude_from_sim no)
@@
 		(fields_autoplaced yes)
 		(property "Reference" "#PWR04"
-			(at 34.29 110.49 0)
+			(at 34.29 115.57 0)
 			(effects
 				(font
@@
 		)
 		(property "Value" "GND"
-			(at 34.29 109.22 0)
+			(at 34.29 114.3 0)
 			(effects
 				(font
@@
 		)
 		(property "Footprint" ""
-			(at 34.29 104.14 0)
+			(at 34.29 109.22 0)
 			(effects
 				(font
@@
 		)
 		(property "Datasheet" ""
-			(at 34.29 104.14 0)
+			(at 34.29 109.22 0)
 			(effects
 				(font
@@
 		)
 		(property "Description" "Power symbol creates a global label with name \"GND\" , ground"
-			(at 34.29 104.14 0)
+			(at 34.29 109.22 0)
 			(effects
 				(font
